Commit message: Hardware interface ready- displaying controllers and HIs succesfully

File: example_2/description/ros2_control/diffbot.ros2_control.xacro (robot description, xacro)
@@ -1,19 +1,12 @@
 <?xml version="1.0"?>
 <robot xmlns:xacro="http://www.ros.org/wiki/xacro">
-  <xacro:macro name="diffbot_ros2_control" params="name prefix use_mock_hardware">
+  <xacro:macro name="diffbot_ros2_control" params="name prefix">
     <ros2_control name="${name}" type="system">
-      <xacro:unless value="${use_mock_hardware}">
         <hardware>
           <plugin>ros2_control_demo_example_2/DiffBotSystemHardware</plugin>
-          <param name="example_param_hw_start_duration_sec">0</param>
-          <param name="example_param_hw_stop_duration_sec">3.0</param>
+          <param name="left_wheel_name">left_wheel_joint</param>
+          <param name="right_wheel_name">drive_r_joint</param>
+          <param name="enc_counts_per_rev">366</param>
         </hardware>
-      </xacro:unless>
-      <xacro:if value="${use_mock_hardware}">
-        <hardware>
-          <plugin>mock_components/GenericSystem</plugin>
-          <param name="calculate_dynamics">true</param>
-        </hardware>
-      </xacro:if>
       <joint name="${prefix}left_wheel_joint">
         <command_interface name="velocity"/>
