Commit message: Added and configured slam_toolbox params and made a map

File: amr_urdf_v3/urdf/amr_urdf_v3.urdf (robot description, URDF)
Before this commit: robot amr_urdf_v3, 10 links, 9 joints
Joints:
- joint left_motor_joint: axis -1 0 0 -> 1 0 0

Commit message: odom glitching?

File: amr_urdf_v3/urdf/amr_urdf_v3.urdf (robot description, URDF)
Before this commit: robot amr_urdf_v3, 10 links, 9 joints
Joints:
- joint imu_joint: origin xyz=0 0 0.148 rpy=0 0 0 -> xyz=0 0 0 rpy=0 0 0
- joint lidar_joint: origin xyz=0.00699999999889178 0 0.25549999999896 rpy=0 0 0 -> xyz=0.00699999999889178 0 0.25549999999896 rpy=0 0 3.1416
